File: Hardware/Motor_Driver/Motor_Driver.kicad_sch (KiCad schematic)
At the start: 71 parts

Commit message: Selected components
Parts:
- removed C? (x2): 470u, symbol Device:C_Small
- removed Q? (x2): Q_NPN_BCE, symbol Device:Q_NPN_BCE
- removed R? (x2): 10k, symbol Device:R_Small
- added Q8: Q_Dual_NPN_NPN_BRT_E1B1C2E2B2C1, Package_TO_SOT_SMD:SOT-363_SC-70-6_Handsoldering, symbol Device:Q_Dual_NPN_NPN_BRT_E1B1C2E2B2C1
- added SW3: SW_DIP_x01, Button_Switch_SMD:SW_DIP_SPSTx01_Slide_6.7x4.1mm_W8.61mm_P2.54mm_LowProfile, symbol Switch:SW_DIP_x01
- C1, C10: renamed from C?; footprint (none) -> Capacitor_SMD:CP_Elec_10x12.6; Part Number (none) -> PCR1E471MCL1GS
- C11, C3, C9: renamed from C?; footprint (none) -> Capacitor_SMD:C_0402_1005Metric_Pad0.74x0.62mm_HandSolder; Part Number (none) -> CL05A104KA5NNNC
- C14, C15: renamed from C?; footprint (none) -> Capacitor_SMD:C_0201_0603Metric_Pad0.64x0.40mm_HandSolder; Part Number (none) -> CL03A105MQ3CSNC
- C2, C5: renamed from C?; footprint (none) -> Capacitor_SMD:C_0805_2012Metric_Pad1.18x1.45mm_HandSolder; Part Number (none) -> CL21A106KOQNNNG
- C4, C6, C7, C8: renamed from C?; footprint (none) -> Capacitor_SMD:C_0805_2012Metric_Pad1.18x1.45mm_HandSolder; Part Number (none) -> CL21A475KBQNNNE
- D1, D2, D3, D4, D6, D7: renamed from D?; value SS10PH10 -> SBRD10200; footprint (none) -> Package_TO_SOT_SMD:TO-252-2; Part Number (none) -> SBRD10200
- D5: renamed from D?; value V8PA10 -> SBRD10200; footprint (none) -> Package_TO_SOT_SMD:TO-252-2; Part Number (none) -> SBRD10200
- D8: renamed from D?; value LED_Small -> Red; footprint (none) -> LED_SMD:LED_0603_1608Metric_Pad1.05x0.95mm_HandSolder; Part Number (none) -> SML-D12U1WT86
- J1: renamed from J?; footprint (none) -> TerminalBlock_MetzConnect:TerminalBlock_MetzConnect_Type701_RT11L03HGLU_1x03_P6.35mm_Horizontal; Part Number (none) -> 796740-3
- J2: renamed from J?; footprint (none) -> Connector_PinHeader_2.54mm:PinHeader_1x05_P2.54mm_Vertical; Part Number (none) -> 61300511121
- J3: renamed from J?; footprint (none) -> Connector_PinHeader_2.54mm:PinHeader_1x06_P2.54mm_Vertical; Part Number (none) -> PPTC061LFBN-RC
- J4: renamed from J?; footprint (none) -> TerminalBlock_MetzConnect:TerminalBlock_MetzConnect_Type701_RT11L02HGLU_1x02_P6.35mm_Horizontal; Part Number (none) -> 1714955
- L1: renamed from L?; footprint (none) -> Inductor_SMD:L_Wuerth_WE-PD-Typ-LS_Handsoldering; Part Number (none) -> 744771147
- Q1, Q2, Q3, Q4, Q5, Q6, Q7: renamed from Q?; footprint (none) -> Package_TO_SOT_SMD:TO-252-2; Part Number (none) -> TSM900N10CP ROG
- R1, R15, R19, R2, R20, R3, R4, R5, R6: renamed from R?; footprint (none) -> Resistor_SMD:R_0201_0603Metric_Pad0.64x0.40mm_HandSolder; Part Number (none) -> RMCF0201FT10K0
- R10, R11, R12, R7, R8, R9: renamed from R?; footprint (none) -> Resistor_SMD:R_0402_1005Metric_Pad0.72x0.64mm_HandSolder; Part Number (none) -> CPF0402B4R0E1
- R13: renamed from R?; value 10k -> 1k; footprint (none) -> Resistor_SMD:R_0201_0603Metric_Pad0.64x0.40mm_HandSolder; Part Number (none) -> RC0201FR-071KL
- R14: renamed from R?; value 20R -> Brake; footprint (none) -> TerminalBlock_MetzConnect:TerminalBlock_MetzConnect_Type701_RT11L02HGLU_1x02_P6.35mm_Horizontal; Part Number HS50 20R J -> 1714955
- R18: renamed from R?; footprint (none) -> Resistor_SMD:R_0603_1608Metric_Pad0.98x0.95mm_HandSolder; Part Number (none) -> WR06X471 JTL
- R21: renamed from R?; footprint (none) -> Resistor_THT:R_Axial_DIN0204_L3.6mm_D1.6mm_P5.08mm_Horizontal; Part Number (none) -> CF18JT120R
- RV1, RV2: renamed from RV?; footprint (none) -> Potentiometer_THT:Potentiometer_Bourns_3266W_Vertical; Part Number (none) -> 3266W-1-503LF
- SW1, SW2: renamed from SW?; footprint (none) -> Button_Switch_SMD:SW_SPST_TL3305A; Part Number (none) -> TL3305AF160QG
- U1: renamed from U?; footprint (none) -> Package_TO_SOT_SMD:TO-252-2; Part Number (none) -> NCP1117DT33T5G
- U2: renamed from U?; footprint (none) -> Package_SO:TSSOP-20_4.4x6.5mm_P0.65mm; Part Number (none) -> DRV8300DIPWR
- U3: renamed from U?; footprint (none) -> Package_TO_SOT_SMD:TO-263-5_TabPin3; Part Number (none) -> TS2596CM550 RNG
- U4: renamed from U?; footprint (none) -> Package_SO:SOIC-8_3.9x4.9mm_P1.27mm; Part Number (none) -> TMCS1108A2BQDR
- U5: renamed from U?; footprint (none) -> Package_SO:SOIC-8_3.9x4.9mm_P1.27mm; Part Number (none) -> LM393ADR
- U7: renamed from U?; footprint (none) -> Package_SO:SOP-8_3.9x4.9mm_P1.27mm; Part Number (none) -> SN65HVD252D
- gave numbers to parts that had none: 1
Connections:
- net +3V3: now also SW3.2; no longer R13.1
- net BRAKE_CON: now also R13.1; no longer Q7.1 (G), R13.2
- net DTR: now also Q8.1 (E1), Q8.5 (B1)
- net EN: now also Q8.3 (C1)
- net IO0: now also Q8.6 (C1)
- net RTS: now also Q8.2 (B1), Q8.4 (E1)
- new net: Q7.1 (G), R13.2, SW3.1
